File: PDB_v2/PD_Board_v2/PD_Board_v2.kicad_sch (KiCad schematic)
At the start: 2 parts, among them J1 Conn_01x03, J2 Conn_01x03

Commit message: 'Completed' Board v2
Parts:
- removed J1, J2: Conn_01x03, symbol Connector_Generic:Conn_01x03
- added H1, H2: MountingHole, MountingHole:MountingHole_3.2mm_M3_Pad, symbol Mechanical:MountingHole
- added J1, J2, J3, J4: ~, Connectors:MR30, symbol Connectors:MR30
- added J5, J6: Conn_01x03_Socket, Connector_PinSocket_2.54mm:PinSocket_1x03_P2.54mm_Vertical, symbol Connector:Conn_01x03_Socket
- added T1: ~, Connectors:XT30, symbol CustomSymbols:XT30
Connections:
- new net: J1.1, J6.3 (Pin_3)
- new net: J1.2, J2.2, J3.2, J4.2, J6.1 (Pin_1), T1.2 (-)
- new net: J1.3, J2.3, J3.3, J4.3, J5.1 (Pin_1), T1.1 (+)
- new net: J3.1, J6.2 (Pin_2)
- new net: J4.1, J5.2 (Pin_2)
- new net: J2.1, J5.3 (Pin_3)
