File: PDB_v3/PD_Board_v3/PD_Board_v3.kicad_sch (KiCad schematic)
At the start: 0 parts

Commit message: started the board
Parts:
- added J1: Wepon, Connectors:MR30, symbol Connector:Conn_01x03_Pin
- added J2: Servo, Connector_PinHeader_2.54mm:PinHeader_1x03_P2.54mm_Vertical, symbol Connector:Conn_01x03_Pin
- added J3: Batt, Connectors:XT30, symbol Connector:Conn_01x02_Pin
- added J4: Drive_pwr, Connectors:XT30, symbol Connector:Conn_01x02_Pin
- added J5: Recv, Connector_PinHeader_2.54mm:PinHeader_2x06_P2.54mm_Horizontal, symbol Connector_Generic:Conn_02x06_Top_Bottom
- added J6: SW, symbol Connector:Conn_01x02_Pin
- added J7: Drive_Sig/5v, Connector_PinHeader_2.54mm:PinHeader_1x04_P2.54mm_Vertical, symbol Connector:Conn_01x04_Pin
Connections:
- new net: J1.1 (Pin_1), J5.7 (Pin_7)
- new net: J1.2 (Pin_2), J4.2 (Pin_2), J6.1 (Pin_1)
- new net: J2.1 (Pin_1), J5.12 (Pin_12)
- new net: J5.4 (Pin_4), J7.1 (Pin_1)
- new net: J5.5 (Pin_5), J7.2 (Pin_2)
- new net: J5.1 (Pin_1), J7.3 (Pin_3)
- new net: J5.6 (Pin_6), J7.4 (Pin_4)
- new net: J3.1 (Pin_1), J6.2 (Pin_2)
- new net BATT+: J1.3 (Pin_3), J3.2 (Pin_2), J4.1 (Pin_1)

Commit message: inital route
Parts:
- added C1: 33pF, Capacitor_SMD:C_0805_2012Metric_Pad1.18x1.45mm_HandSolder, symbol Device:C_Small
- added C2: 10uF, Capacitor_SMD:C_0805_2012Metric_Pad1.18x1.45mm_HandSolder, symbol Device:C_Small
- added C3, C5: 100nF, Capacitor_SMD:C_0805_2012Metric_Pad1.18x1.45mm_HandSolder, symbol Device:C_Small
- added C4: 47uF, Capacitor_SMD:C_0805_2012Metric_Pad1.18x1.45mm_HandSolder, symbol Device:C_Small
- added H1, H3, H4: MountingHole, MountingHole:MountingHole_3.5mm, symbol Mechanical:MountingHole
- added J8: DR_L, Connectors:MR30, symbol Connector:Conn_01x03_Pin
- added J9: DR_R, Connectors:MR30, symbol Connector:Conn_01x03_Pin
- added L1: 3.3uH, Inductor_SMD:L_Coilcraft_XAL7070-XXX, symbol Device:L_Small
- added R1: 100k, Resistor_SMD:R_0805_2012Metric_Pad1.20x1.40mm_HandSolder, symbol Device:R_Small_US
- added R2: 270k, Resistor_SMD:R_0805_2012Metric_Pad1.20x1.40mm_HandSolder, symbol Device:R_Small_US
- added R3: 12.1k, Resistor_SMD:R_0805_2012Metric_Pad1.20x1.40mm_HandSolder, symbol Device:R_Small_US
- added R4: 30k, Resistor_SMD:R_0805_2012Metric_Pad1.20x1.40mm_HandSolder, symbol Device:R_Small_US
- added U1: ~, Package_TO_SOT_SMD:SOT-23-6, symbol Project:TPS565247DRL
- J3: renamed from J6; footprint (none) -> Project:SMD_SW
- J7: renamed from J2; footprint Connector_PinHeader_2.54mm:PinHeader_1x03_P2.54mm_Vertical -> Connectors:MR30
- renumbered J3 to J2, J7 to J4, J4 to J6
Connections:
- net +BATT_SW: now reaches J1.1 (Pin_1)
- net +BATT_SW: now also J3.2 (Pin_2), J6.1 (Pin_1), C2.1, C3.1, R1.1, U1.1 (VIN); no longer J5.7 (Pin_7)
- net +6V: now reaches J7.1 (Pin_1)
- net +6V: now also C1.1, C4.1, C5.1, L1.2, R2.1; no longer J5.12 (Pin_12)
- net S1: now reaches J7.2 (Pin_2)
- net S1: now also J5.1 (Pin_1)
- net GND: now reaches J7.3 (Pin_3)
- net GND: now also J1.3 (Pin_3), J2.2 (Pin_2), J4.1 (Pin_1), J5.10 (Pin_10), J5.3 (Pin_3), J5.4 (Pin_4), J5.9 (Pin_9), J6.2 (Pin_2), C2.2, C3.2, C4.2, C5.2, R3.2, R4.2, U1.3 (GND), U1.4 (AGND)
- net +5V: now reaches J4.2 (Pin_2), J5.5 (Pin_5)
- net +5V: now also J5.11 (Pin_11), J5.2 (Pin_2), J5.8 (Pin_8)
- net S3: now reaches J4.3 (Pin_3)
- net S3: now also J5.7 (Pin_7); no longer J5.1 (Pin_1)
- net S2: now reaches J5.6 (Pin_6)
- net S2: now also J1.2 (Pin_2); no longer J4.4 (Pin_4)
- net +BATT: now reaches J2.1 (Pin_1)
- net +BATT: now also J3.1 (Pin_1); no longer J3.2 (Pin_2)
- removed net BATT+: J1.3 (Pin_3), J2.2 (Pin_2), J6.1 (Pin_1)
- new net: R1.2, R3.1, U1.5 (EN)
- new net: C1.2, R2.2, R4.1, U1.6 (FB)
- new net: L1.1, U1.2 (SW)
- new net S4: J4.4 (Pin_4), J5.12 (Pin_12)
Other:
- moved on the sheet: J1, J2, J3, J4, J5, J6, J7

Commit message: almost done
Parts:
- removed J4: Drive_Sig/5v, Connector_PinHeader_2.54mm:PinHeader_1x04_P2.54mm_Vertical, symbol Connector:Conn_01x04_Pin
- removed J6: Drive_pwr, Connectors:XT30, symbol Connector:Conn_01x02_Pin
- removed J8: DR_L, Connectors:MR30, symbol Connector:Conn_01x03_Pin
- removed J9: DR_R, Connectors:MR30, symbol Connector:Conn_01x03_Pin
- added C6: 10uF, Capacitor_SMD:C_0603_1608Metric_Pad1.08x0.95mm_HandSolder, symbol Device:C_Small
- added E1: Dual_ESC, Project:Dual_ESC, symbol Project:Dual_ESC
- C1: Part # (none) -> 399-C0805C330J3HACTUCT-ND
- C2: footprint Capacitor_SMD:C_0805_2012Metric_Pad1.18x1.45mm_HandSolder -> Capacitor_SMD:C_0603_1608Metric_Pad1.08x0.95mm_HandSolder; Part # (none) -> 445-9015-1-ND
- C3, C5: Part # (none) -> 399-C0805F104K1RACAUTOCT-ND
- C4: footprint Capacitor_SMD:C_0805_2012Metric_Pad1.18x1.45mm_HandSolder -> Capacitor_SMD:C_1210_3225Metric_Pad1.33x2.70mm_HandSolder; Part # (none) -> 490-6539-1-ND
- J1, J2, J3, J5, J7: now not fitted
- L1: footprint Inductor_SMD:L_Coilcraft_XAL7070-XXX -> Project:Inductor; Part # (none) -> 2037-VAMV1009AA-3R3MM2CT-ND
- R1: Part # (none) -> P100KDACT-ND
- R2: Part # (none) -> P270KDACT-ND
- R3: Part # (none) -> P12.1KDACT-ND
- R4: Part # (none) -> P30KDACT-ND
- U1: Part # (none) -> 296-TPS565247DRLRCT-ND
Connections:
- net +5V: now also E1.4 (5v)
- net +BATT_SW: now also C6.1, E1.1 (BATT+)
- net GND: now also C6.2, E1.2 (BATT-), E1.3 (GND)
- net S3: now also E1.5 (S0)
- net S4: now also E1.6 (S1)
- no-connect marks 0 -> 6
Other:
- moved on the sheet: H1, H3, H4
